Commit message: backport to ros1

File: odrive_botwheel_explorer/description/urdf/diffbot.ros2_control.xacro (robot description, xacro)
@@ -1,9 +1,9 @@
 <?xml version="1.0"?>
 <robot xmlns:xacro="http://www.ros.org/wiki/xacro">
-  <xacro:macro name="diffbot_ros2_control" params="name prefix use_mock_hardware">
+  <xacro:macro name="diffbot_ros_control" params="name prefix use_mock_hardware">
     <ros2_control name="${name}" type="system">
       <xacro:unless value="${use_mock_hardware}">
         <hardware>
-          <plugin>odrive_ros2_control_plugin/ODriveHardwareInterface</plugin>
+          <plugin>odrive_ros_control_plugin/ODriveHardwareInterface</plugin>
           <param name="can">can0</param>
         </hardware>
